Commit message: last commit

File: anymal_c_simple_description/urdf/old.urdf (robot description, URDF)
Before this commit: robot anymal, 84 links, 83 joints
Links:
- removed link rot_y
- removed link rot_z
- removed link trans_x
- removed link trans_y
- removed link trans_z
Joints:
- removed joint rot_y_to_rot_torso
- removed joint rot_z_to_rot_y
- removed joint trans_x_to_trans_y
- removed joint trans_y_to_trans_z
- removed joint trans_z_to_rot_z
- removed joint world_to_trans_x
- added joint base_joint: type floating, parent base_link, child Torso, origin xyz=0 0 0 rpy=0 0 0
