Commit message: ultimo commit

File: anymal_c_simple_description/urdf/anymal.urdf (robot description, URDF)
Before this commit: robot anymal, 78 links, 77 joints
Links:
- removed link base_inertia
- link base: mass None -> 6.222
Joints:
- removed joint base_to_base_inertia

File: anymal_c_simple_description/urdf/model.urdf (robot description, URDF)
Before this commit: robot anymal, 84 links, 83 joints
Links:
- removed link Torso
- removed link base_inertia
- removed link base_link
- removed link rot_y
- removed link rot_z
- removed link trans_x
- removed link trans_y
- removed link trans_z
- added link base, mass 3.222; collision box size=0.58 0.14 0.18; collision cylinder length=0.145 radius=0.09
Joints:
- removed joint base_to_base_inertia
- removed joint rot_y_to_rot_torso
- removed joint rot_z_to_rot_y
- removed joint trans_x_to_trans_y
- removed joint trans_y_to_trans_z
- removed joint trans_z_to_rot_z
- removed joint world_to_trans_x
- joint base_LF_HAA: parent Torso -> base
- joint base_LH_HAA: parent Torso -> base
- joint base_RF_HAA: parent Torso -> base
- joint base_RH_HAA: parent Torso -> base
- joint base_battery: parent Torso -> base
- joint base_bottom_shell: parent Torso -> base
- joint base_face_front: parent Torso -> base
- joint base_face_rear: parent Torso -> base
- joint base_handle: parent Torso -> base
- joint base_hatch: parent Torso -> base
- joint base_remote: parent Torso -> base
- joint base_to_depth_camera_left_camera: parent Torso -> base
- joint base_to_depth_camera_right_camera: parent Torso -> base
- joint base_to_docking_hatch_cover: parent Torso -> base
- joint base_to_lidar_cage: parent Torso -> base
- joint base_top_shell: parent Torso -> base
- joint imu_joint: parent Torso -> base
