Commit message: last commit

File: anymal_c_simple_description/urdf/model2.urdf (robot description, URDF)
Before this commit: robot anymal, 77 links, 76 joints
Links:
- removed link base_link
- added link base, mass 6.222; collision box size=0.58 0.14 0.18; collision cylinder length=0.145 radius=0.09
Joints:
- joint base_LF_HAA: parent base_link -> base
- joint base_LH_HAA: parent base_link -> base
- joint base_RF_HAA: parent base_link -> base
- joint base_RH_HAA: parent base_link -> base
- joint base_battery: parent base_link -> base
- joint base_bottom_shell: parent base_link -> base
- joint base_face_front: parent base_link -> base
- joint base_face_rear: parent base_link -> base
- joint base_handle: parent base_link -> base
- joint base_hatch: parent base_link -> base
- joint base_remote: parent base_link -> base
- joint base_to_depth_camera_left_camera: parent base_link -> base
- joint base_to_depth_camera_right_camera: parent base_link -> base
- joint base_to_docking_hatch_cover: parent base_link -> base
- joint base_to_lidar_cage: parent base_link -> base
- joint base_top_shell: parent base_link -> base
- joint imu_joint: parent base_link -> base
